Commit message: Basic gripper operation added

File: myrobot/model/robot_model.urdf (robot description, URDF)
Before this commit: robot myrobot, 11 links, 10 joints
Links:
- removed link camera_link_optical
- link link_camera: geometry collision box size=0.02 0.07 0.04; visual box size=0.02 0.07 0.04
Joints:
- removed joint camera_optical_joint

File: myrobot/model/robot_model.xacro (robot description, xacro)
@@ -193,5 +193,5 @@
             <origin xyz="0.0 0.0 0.0"/>
             <geometry>
-                <box size="0.02 0.04 0.04"/>
+                <box size="0.02 0.07 0.04"/>
             </geometry>
             <material name="red"/>
@@ -200,5 +200,5 @@
             <origin xyz="0.0 0.0 0.0"/>
             <geometry>
-                <box size="0.02 0.04 0.04"/>
+                <box size="0.02 0.07 0.04"/>
             </geometry>
         </collision>
@@ -302,13 +302,4 @@
         <dynamics damping="0.7" friction="0.7"/>
     </joint>
-    <!--joint and link for camera-->
-    <joint name="camera_optical_joint" type="fixed">
-          <origin xyz="0 0 0" rpy="${-pi/2} 0 ${-pi/2}"/>
-          <!-- <origin xyz="0 0.1 0" rpy="0 ${-pi/2} 0"/> -->
-          <parent link="link_camera"/>
-          <child link="camera_link_optical"/>
-    </joint>
-    <link name="camera_link_optical">
-    </link>
     <!--ros2_control module-->
     <ros2_control name="GazeboSystem" type="system">
@@ -381,68 +372,66 @@
     <!--plugin for camera-->
     <gazebo reference="link_camera">
-      <sensor type="camera" name="camera1">
-        <update_rate>30.0</update_rate>
-        <camera name="head">
-          <horizontal_fov>1.3962634</horizontal_fov>
-          <image>
-            <width>800</width>
-            <height>800</height>
-            <format>R8G8B8</format>
-          </image>
-          <clip>
-            <near>0.02</near>
-            <far>300</far>
-          </clip>
-          <noise>
-            <type>gaussian</type>
-            <!-- Noise is sampled independently per pixel on each frame.
-            That pixel's noise value is added to each of its color
-            channels, which at that point lie in the range [0,1]. -->
-            <mean>0.0</mean>
-            <stddev>0.007</stddev>
-          </noise>
-        </camera>
-        <plugin name="camera_controller" filename="libgazebo_ros_camera.so">
-          <alwaysOn>true</alwaysOn>
-          <updateRate>0.0</updateRate>
-          <cameraName>myrobot/camera1</cameraName>
-          <imageTopicName>image_raw</imageTopicName>
-          <cameraInfoTopicName>camera_info</cameraInfoTopicName>
-          <frameName>camera_link_optical</frameName>
-          <!-- setting hackBaseline to anything but 0.0 will cause a misalignment
-          between the gazebo sensor image and the frame it is supposed to
-          be attached to -->
-          <hackBaseline>0.0</hackBaseline>
-          <distortionK1>0.0</distortionK1>
-          <distortionK2>0.0</distortionK2>
-          <distortionK3>0.0</distortionK3>
-          <distortionT1>0.0</distortionT1>
-          <distortionT2>0.0</distortionT2>
-          <CxPrime>0</CxPrime>
-          <Cx>0.0</Cx>
-          <Cy>0.0</Cy>
-          <focalLength>0.0</focalLength>
-        </plugin>
-      </sensor>
-    </gazebo>
-    <!--plugin for vacuum gripper-->
     <!-- <gazebo>
-      <plugin name="gazebo_ros_vacuum_gripper" filename="libgazebo_ros_vacuum_gripper.so">
-        <robotNamespace>/robot_model/link_vacuum</robotNamespace>
-        <bodyName>link_vacuum</bodyName>
-        <topicName>grasping</topicName>
-        <maxForce>50</maxForce>
-        <maxDistance>0.05</maxDistance>
-        <minDistance>0.01</minDistance>
-      </plugin>
-    </gazebo> -->
-    <gazebo>
-      <plugin  name='vacuum_gripper' filename='libgazebo_ros_vacuum_gripper.so'>
-        <ros>
-          <namespace>/robot_model</namespace>
-        </ros>
-        <link_name>link_vacuum</link_name>
-        <maxDistance>0.05</maxDistance>
-      </plugin>
-    </gazebo>
+    <link name= "link_camera"> -->
+    <sensor type="multicamera" name="sensor_name">
+          <camera name="left">
+            <horizontal_fov>1.3962634</horizontal_fov>
+            <image>
+              <width>800</width>
+              <height>800</height>
+              <format>R8G8B8</format>
+            </image>
+            <clip>
+              <near>0.02</near>
+              <far>300</far>
+            </clip>
+            <noise>
+              <type>gaussian</type>
+              <mean>0.0</mean>
+              <stddev>0.007</stddev>
+            </noise>
+          </camera>
+          <camera name="right">
+            <pose>0 -0.07 0 0 0 0</pose>
+            <horizontal_fov>1.3962634</horizontal_fov>
+            <image>
+              <width>800</width>
+              <height>800</height>
+              <format>R8G8B8</format>
+            </image>
+            <clip>
+              <near>0.02</near>
+              <far>300</far>
+            </clip>
+            <noise>
+              <type>gaussian</type>
+              <mean>0.0</mean>
+              <stddev>0.007</stddev>
+            </noise>
+          </camera>
+          <!-- Set update_rate only sensor, not on plugin -->
+          <update_rate>1</update_rate>
+          <plugin name="plugin_name" filename="libgazebo_ros_camera.so">
+            <ros>
+              <namespace>custom_ns</namespace>
+              <!-- topics need to be prefixed with camera_name for remapping -->
+              <argument>custom_camera/left/image_raw:=custom_camera/left/custom_image</argument>
+              <argument>custom_camera/right/image_raw:=custom_camera/right/custom_image</argument>
+              <argument>custom_camera/left/camera_info:=custom_camera/left/custom_camera_info</argument>
+              <argument>custom_camera/right/camera_info:=custom_camera/right/custom_camera_info</argument>
+            </ros>
+            <camera_name>custom_camera</camera_name>
+            <frameName>left_camera_optical_frame</frameName>
+          </plugin>
+        </sensor>
+    </gazebo>
+  <gazebo>
+    <plugin  name='vacuum_gripper' filename='libgazebo_ros_vacuum_gripper.so'>
+      <ros>
+        <namespace>/robot_model</namespace>
+      </ros>
+      <link_name>link_vacuum</link_name>
+      <maxDistance>0.05</maxDistance>
+    </plugin>
+  </gazebo>
 </robot>
