Commit message: setting joint_cameraHolder_camera as revolute type to get camera tf frame

File: myrobot/model/robot_model.xacro (robot description, xacro)
@@ -288,8 +288,12 @@
     </joint>
     <!--joint of link_cameraHolder and link_camera-->
-    <joint name="joint_cameraHolder_camera" type="fixed">
+    <joint name="joint_cameraHolder_camera" type="revolute">
         <parent link="link_cameraHolder"/>
         <child link="link_camera"/>
         <origin xyz="-0.015 0.0 0.035" rpy="0.0 ${-pi/2} 0.0"/>
+        <!-- added for revolute joint type -->
+        <axis xyz="1 0 0"/>
+        <limit effort="1000.0" upper="0.0" lower="0.0" velocity="0.0"/>
+        <dynamics damping="100.0" friction="100.0"/>
     </joint>
     <!--joint of link_gripper and link_vacuum-->
@@ -356,4 +360,14 @@
           <param name="min">-2.0</param>
           <param name="max">2.0</param>
+        </command_interface>
+        <state_interface name="position"/>
+        <state_interface name="velocity"/>
+        <state_interface name="effort"/>
+      </joint>
+      <!-- added for camera revolute joint type -->
+      <joint name="joint_cameraHolder_camera">
+        <command_interface name="position">
+          <param name="min">-0.0</param>
+          <param name="max">0.0</param>
         </command_interface>
         <state_interface name="position"/>

Commit message: 2 new objects added to gazebo, small link for vacuum added

File: myrobot/model/robot_model.xacro (robot description, xacro)
@@ -230,4 +230,26 @@
       <material>Gazebo/Black</material>
     </gazebo>
+    <!-- tcp link -->
+    <link name="link_tcp">
+        <visual>
+            <origin xyz="0.0 0.0 0.0" rpy="0.0 0.0 0.0"/>
+            <geometry>
+                <box size="0.0001 0.0001 0.0001"/>
+            </geometry>
+            <material name="black"/>
+        </visual>
+        <collision>
+            <origin xyz="0.0 0.0 0.0" rpy="0.0 0.0 0.0"/>
+            <geometry>
+                <box size="0.0001 0.0001 0.0001"/>
+            </geometry>
+        </collision>
+        <xacro:default_inertial mass="0.001" w="0.0001" h="0.001"/>
+    </link>
+    <gazebo reference= "link_tcp">
+      <mu1>0.2</mu1>
+      <mu2>0.2</mu2>
+      <material>Gazebo/Black</material>
+    </gazebo>
     <!--joint of world and link_base-->
     <joint name="joint_world_base" type="fixed">
@@ -306,4 +328,13 @@
         <dynamics damping="0.7" friction="0.7"/>
     </joint>
+    <!--joint of link_vacuum and link_tcp-->
+    <joint name="joint_vacuum_tcp" type="revolute">
+        <parent link="link_vacuum"/>
+        <child link="link_tcp"/>
+        <origin xyz="0.0 0.0 0.0" rpy="0.0 0.0 0.0"/>
+        <axis xyz="1 0 0"/>
+        <limit effort="1000.0" upper="2.0" lower="-2.0" velocity="5.0"/>
+        <dynamics damping="0.7" friction="0.7"/>
+    </joint>
     <!--ros2_control module-->
     <ros2_control name="GazeboSystem" type="system">
@@ -367,4 +398,14 @@
       <!-- added for camera revolute joint type -->
       <joint name="joint_cameraHolder_camera">
+        <command_interface name="position">
+          <param name="min">-0.0</param>
+          <param name="max">0.0</param>
+        </command_interface>
+        <state_interface name="position"/>
+        <state_interface name="velocity"/>
+        <state_interface name="effort"/>
+      </joint>
+      <!-- added for tcp revolute joint type -->
+      <joint name="joint_vacuum_tcp">
         <command_interface name="position">
           <param name="min">-0.0</param>
@@ -442,11 +483,12 @@
   <!-- vacuum gripper plugins -->
   <gazebo>
-    <plugin  name='vacuum_gripper1' filename='libgazebo_ros_vacuum_gripper.so'>
-      <ros>
-        <namespace>/robot_model1</namespace>
-      </ros>
-      <link_name>link_vacuum</link_name>
-      <max_distance>0.5</max_distance>
-      <fixed>ground_plane</fixed>
+    <plugin  name='vacuum_gripper' filename='libgazebo_ros_vacuum_gripper.so'>
+      <ros>
+        <namespace>/robot_model</namespace>
+      </ros>
+      <!-- <link_name>link_vacuum</link_name> -->
+      <link_name>link_tcp</link_name>
+      <max_distance>0.3</max_distance> <!--0.5-->
+      <!-- <fixed>ground_plane</fixed> -->
     </plugin>
   </gazebo>
